Commit message: WIP robinzen in mockup

File: xbt_bringup/urdf/a_bot_macro.xacro (robot description, xacro)
@@ -10,5 +10,5 @@
         parent
         transmission_hw_interface:=hardware_interface/PositionJointInterface
-        kinematics_parameters_file:='$(find ur_description)/config/ur5e/default_kinematics.yaml'
+        kinematics_parameters_file:='$(find xbt_bringup)/config/calibration.yaml'
         joint_limits_parameters_file:='$(find ur_description)/config/ur5e/joint_limits.yaml'
         *origin">

File: xbt_bringup/urdf/a_bot_scene.xacro (robot description, xacro)
@@ -4,5 +4,5 @@
         default="$(find ur_description)/config/ur5e/joint_limits.yaml" />
     <xacro:arg name="kinematics_parameters_file"
-        default="$(find ur_description)/config/ur5e/default_kinematics.yaml" />
+        default="$(find xbt_bringup)/config/calibration.yaml" />
     <xacro:arg name="transmission_hw_interface" default="hardware_interface/PositionJointInterface" />
     <xacro:include filename="$(find homestri_description)/urdf/macros/simple_pedestal_macro.xacro" />
@@ -12,5 +12,5 @@
         parent="world"
         height="0.6"
-        radius="0.15"
+        radius="0.2"
     />
     <xacro:a_bot
@@ -21,5 +21,5 @@
         kinematics_parameters_file="$(arg kinematics_parameters_file)"
     >
-        <origin xyz="0 0 0" rpy="0 0 ${pi/2}" />
+        <origin xyz="0 0 0" rpy="0 0 ${-pi/2}" />
     </xacro:a_bot>
     <link name="world" />
