Commit message: finish robinzen, added 3dprinitng open/close oven

File: xbt_bringup/urdf/a_bot_scene.xacro (robot description, xacro)
@@ -28,3 +28,63 @@
         </plugin>
     </gazebo>
+    <link name="wall_1">
+        <collision>
+        <geometry>
+            <box size="0.02 3.5 3.5"/>
+        </geometry>
+        </collision>
+    </link>
+    <link name="wall_2">
+        <collision>
+        <geometry>
+            <box size="3 3 0.02"/>
+        </geometry>
+        </collision>
+    </link>
+    <link name="wall_3">
+        <collision>
+        <geometry>
+            <box size="3 3 0.02"/>
+        </geometry>
+        </collision>
+    </link>
+    <link name="wall_4">
+        <collision>
+        <geometry>
+            <box size="0.02 3 3.5"/>
+        </geometry>
+        </collision>
+    </link>
+    <joint name="wall_1_joint" type="fixed">
+        <parent link="world"/>
+        <child link="wall_1"/>
+        <origin xyz="-0.5 0 0" rpy="0 0 0"/>
+    </joint>
+    <joint name="wall_2_joint" type="fixed">
+        <parent link="world"/>
+        <child link="wall_2"/>
+        <origin xyz="0 0 -0.02" rpy="0 0 0"/>
+    </joint>
+    <joint name="wall_3_joint" type="fixed">
+        <parent link="world"/>
+        <child link="wall_3"/>
+        <origin xyz="0 0 1.5" rpy="0 0 0"/>
+    </joint>
+    <joint name="wall_4_joint" type="fixed">
+        <parent link="world"/>
+        <child link="wall_4"/>
+        <origin xyz="0.7 1.5 0" rpy="0 0 0"/>
+    </joint>
+    <!-- <link name="eef_collision">
+        <collision>
+        <geometry>
+            <box size="0.15 0.03 0.2"/>
+        </geometry>
+        </collision>
+    </link>
+    <joint name="eef_collision_joint" type="fixed">
+        <parent link="wrist_3_link"/>
+        <child link="eef_collision"/>
+        <origin xyz="0 0 0.1" rpy="0 0 0"/>
+    </joint> -->
 </robot>
